File: v0.5.kicad_pcb (KiCad board)
At the start: 2 copper layers, 82 x 38 mm, 65 parts, among them J1 Conn_01x02_Pin, J2 USB_B_Micro, J3 Conn_02x06_Odd_Even, J4 Screw_Terminal_01x08, J5 Screw_Terminal_01x04, J6 Conn_Coaxial_Small, J7 Conn_Coaxial_Small, Q1 MMBT3904, Q2 SiS454DN, Q3 SiS454DN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

Commit message: Updated gerber files
Changed lines of the file:
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@@
 		(tags "LoRa Low Power Long Range Transceiver Module")
 		(property "Reference" "U8"
-			(at 0 9.2 90)
+			(at -2.45 0 180)
 			(layer "B.SilkS")
 			(effects
@@
 	)
 	(gr_text "GND"
-		(at 159.7 103.6 0)
+		(at 160.4 103.6 0)
 		(layer "F.SilkS")
 		(effects
@@
 	)
 	(gr_text "Flight Computer v0.5\nTim Drake"
-		(at 97.7 110.9 -0)
-		(layer "F.SilkS")
-		(effects
+		(at 97.6 110.6 -0)
+		(layer "F.SilkS")
+		(effects
